File: PLC4UNI-GC1_PCB/IN-4-20MA.kicad_sch (KiCad schematic)
At the start: 8 parts

Commit message: Actualizacion a la fecha
Other:
- moved on the sheet: R27, R9
Changed lines of the file:
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@@
 	(paper "A4")
 	(junction
-		(at 127 81.28)
+		(at 120.65 81.28)
 		(diameter 0)
 		(color 0 0 0 0)
@@
 	)
 	(junction
+		(at 137.16 81.28)
+		(diameter 0)
+		(color 0 0 0 0)
+	)
+	(junction
 		(at 200.66 81.28)
 		(diameter 0)
@@
 	)
 	(junction
-		(at 137.16 81.28)
-		(diameter 0)
-		(color 0 0 0 0)
-	)
-	(junction
 		(at 137.16 107.95)
 		(diameter 0)
@@
 	)
 	(junction
-		(at 127 107.95)
+		(at 120.65 107.95)
 		(diameter 0)
 		(color 0 0 0 0)
@@
 	(wire
 		(pts
-			(xy 127 81.28) (xy 137.16 81.28)
+			(xy 120.65 81.28) (xy 137.16 81.28)
 		)
 		(stroke
@@
 	(wire
 		(pts
-			(xy 123.19 81.28) (xy 127 81.28)
+			(xy 116.84 81.28) (xy 120.65 81.28)
 		)
 		(stroke
@@
 	(wire
 		(pts
-			(xy 137.16 107.95) (xy 127 107.95)
+			(xy 137.16 107.95) (xy 120.65 107.95)
 		)
 		(stroke
@@
 	(wire
 		(pts
-			(xy 110.49 107.95) (xy 127 107.95)
-		)
-		(stroke
-			(width 0)
-			(type default)
-		)
-	)
-	(wire
-		(pts
-			(xy 110.49 81.28) (xy 115.57 81.28)
+			(xy 104.14 107.95) (xy 120.65 107.95)
+		)
+		(stroke
+			(width 0)
+			(type default)
+		)
+	)
+	(wire
+		(pts
+			(xy 104.14 81.28) (xy 109.22 81.28)
 		)
 		(stroke
@@
 	(wire
 		(pts
-			(xy 127 102.87) (xy 127 107.95)
-		)
-		(stroke
-			(width 0)
-			(type default)
-		)
-	)
-	(wire
-		(pts
-			(xy 127 81.28) (xy 127 95.25)
+			(xy 120.65 102.87) (xy 120.65 107.95)
+		)
+		(stroke
+			(width 0)
+			(type default)
+		)
+	)
+	(wire
+		(pts
+			(xy 120.65 81.28) (xy 120.65 95.25)
 		)
 		(stroke
@@
 	(hierarchical_label "IN_P"
 		(shape input)
-		(at 110.49 81.28 180)
+		(at 104.14 81.28 180)
 		(effects
 			(font
@@
 	(hierarchical_label "IN_N"
 		(shape input)
-		(at 110.49 107.95 180)
+		(at 104.14 107.95 180)
 		(effects
 			(font
@@
 	(symbol
 		(lib_id "Resistor_US_AKL:R_0805")
-		(at 127 99.06 180)
+		(at 120.65 99.06 180)
 		(unit 1)
 		(body_style 1)
@@
 		(dnp no)
 		(property "Reference" "R9"
-			(at 128.524 96.7739 0)
+			(at 122.174 96.7739 0)
 			(show_name no)
 			(do_not_autoplace no)
@@
 		)
 		(property "Value" "120R"
-			(at 128.524 99.3139 0)
+			(at 122.174 99.3139 0)
 			(show_name no)
 			(do_not_autoplace no)
@@
 		)
 		(property "Footprint" "Resistor_SMD_AKL:R_0805_2012Metric"
-			(at 127 87.63 0)
+			(at 120.65 87.63 0)
 			(hide yes)
 			(show_name no)
@@
 		)
 		(property "Datasheet" ""
-			(at 127 99.06 0)
+			(at 120.65 99.06 0)
 			(hide yes)
 			(show_name no)
@@
 		)
 		(property "Description" "SMD 0805 Chip Resistor, US Symbol, Alternate KiCad Library"
-			(at 127 99.06 0)
+			(at 120.65 99.06 0)
 			(hide yes)
 			(show_name no)
@@
 		)
 		(property "TOL" "0.1%"
-			(at 130.81 101.6 0)
+			(at 124.46 101.6 0)
 			(show_name no)
 			(do_not_autoplace no)
@@
 	(symbol
 		(lib_id "Resistor_US_AKL:R_0805")
-		(at 119.38 81.28 270)
+		(at 113.03 81.28 270)
 		(unit 1)
 		(body_style 1)
@@
 		(dnp no)
 		(property "Reference" "R27"
-			(at 117.094 80.01 90)
+			(at 110.744 80.01 90)
 			(show_name no)
 			(do_not_autoplace no)
@@
 		)
 		(property "Value" "49.9R"
-			(at 121.666 83.566 90)
+			(at 115.316 83.566 90)
 			(show_name no)
 			(do_not_autoplace no)
@@
 		)
 		(property "Footprint" "Resistor_SMD_AKL:R_0805_2012Metric"
-			(at 107.95 81.28 0)
+			(at 101.6 81.28 0)
 			(hide yes)
 			(show_name no)
@@
 		)
 		(property "Datasheet" ""
-			(at 119.38 81.28 0)
+			(at 113.03 81.28 0)
 			(hide yes)
 			(show_name no)
@@
 		)
 		(property "Description" "SMD 0805 Chip Resistor, US Symbol, Alternate KiCad Library"
-			(at 119.38 81.28 0)
+			(at 113.03 81.28 0)
 			(hide yes)
 			(show_name no)
@@
 		)
 		(property "TOL" "0.1%"
-			(at 124.206 80.01 90)
-			(show_name no)
-			(do_not_autoplace no)
+			(at 117.856 80.01 90)
+			(show_name no)
+			(do_not_autoplace no)
