File: PLC4UNI-GC1_PCB/IN-DI.kicad_sch (KiCad schematic)
At the start: 6 parts, among them U5 AT3H4B-CUH-S

Commit message: Actualizacion a la fecha
Parts:
- added LED8: LED_0603_Red, LED_SMD_AKL:LED_0603_1608Metric, symbol LED_AKL:LED_0603_Red
- added R67: R_0603, Resistor_SMD_AKL:R_0603_1608Metric, symbol Resistor_US_AKL:R_0603
Connections:
- net +3.3V: now also R67.1
- net OUT: now also LED8.1 (K)
- new net: LED8.2 (A), R67.2
Other:
- note added: "Entrada 5V a 24V"
- moved on the sheet: R16
