File: PLC4UNI-GC1_PCB/OUT-4-20MA.kicad_sch (KiCad schematic)
At the start: 11 parts, among them Q1 NCE60P04R, U8 GP8302-TC50-EW

Commit message: Actualizacion a la fecha
Connections:
- net +24V renamed VDC
Changed lines of the file:
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@@
 	)
 	(symbol
-		(lib_id "power:+24V")
+		(lib_id "power:VDC")
 		(at 127 82.55 0)
 		(unit 1)
@@
 		(dnp no)
 		(fields_autoplaced yes)
-		(property "Reference" "#PWR031"
+		(property "Reference" "#PWR0113"
 			(at 127 86.36 0)
 			(hide yes)
@@
 			)
 		)
-		(property "Value" "+24V"
+		(property "Value" "VDC"
 			(at 127 77.47 0)
 			(show_name no)
@@
 			)
 		)
-		(property "Description" "Power symbol creates a global label with name \"+24V\""
+		(property "Description" "Power symbol creates a global label with name \"VDC\""
 			(at 127 82.55 0)
 			(hide yes)
@@
 			(project "PLC4UNI-GC1"
 				(path "/78be00cd-daf6-4f2a-9977-d3085e20b798/ca21e56d-4223-44eb-9b60-6c8fe421c362/b87f0d40-2256-4199-83d6-86177a261c42"
-					(reference "#PWR031")
+					(reference "#PWR0113")
 					(unit 1)
 				)
@@
 	)
 	(symbol
-		(lib_id "power:+24V")
+		(lib_id "power:VDC")
 		(at 184.15 76.2 0)
 		(unit 1)
@@
 		(dnp no)
 		(fields_autoplaced yes)
-		(property "Reference" "#PWR034"
+		(property "Reference" "#PWR0112"
 			(at 184.15 80.01 0)
 			(hide yes)
@@
 			)
 		)
-		(property "Value" "+24V"
+		(property "Value" "VDC"
 			(at 184.15 71.12 0)
 			(show_name no)
@@
 			)
 		)
-		(property "Description" "Power symbol creates a global label with name \"+24V\""
+		(property "Description" "Power symbol creates a global label with name \"VDC\""
 			(at 184.15 76.2 0)
 			(hide yes)
@@
 			(project "PLC4UNI-GC1"
 				(path "/78be00cd-daf6-4f2a-9977-d3085e20b798/ca21e56d-4223-44eb-9b60-6c8fe421c362/b87f0d40-2256-4199-83d6-86177a261c42"
-					(reference "#PWR034")
-					(unit 1)
-				)
+					(reference "#PWR0112")
+					(unit 1)
+				)
