File: PLC4UNI-GC1_PCB/PLC4UNI-GC1.kicad_sch (KiCad schematic)
At the start: 6 parts

Commit message: Actualizacion a la fecha
Parts:
- renumbered connector-up1 to J2, connector-up2 to J3, connector-down1 to J4, connector-down2 to J5
Connections:
- net control/CON_OUT_NPN1: now also J4.3; no longer J4.4
- net control/CON_OUT_NPN2: now also J4.4; no longer J4.5
- net control/CON_OUT_NPN3: now also J4.5; no longer J4.6
- net control/CON_OUT_NPN4: now also J4.6; no longer J4.7
- net control/CON_OUT_PNP1: now also J4.1; no longer J4.8
- net control/CON_OUT_PNP2: now also J4.2; no longer J4.9
- net control/CON_RS485_A: now also J4.9; no longer J4.2
- net control/CON_RS485_B: now also J4.8; no longer J4.3
- net control/CON_RS485_G: now also J4.7; no longer J4.1
