File: PLC4UNI-GC1_PCB/PowerSupply.kicad_sch (KiCad schematic)
At the start: 16 parts, among them U3 AP63203WU

Commit message: Actualizacion a la fecha
Parts:
- removed C41: 47UF, Capacitor_SMD:CP_Elec_6.3x7.7, symbol MG_CAPACITOR:CAP-POL-SMD-47UF-16V-D6.3MM
- removed D1, D2: SS14, Diode_SMD:D_SMA, symbol Diode:SS14
- removed L1: 10uH, Inductor_SMD:L_APV_APH0630, symbol Device:L_Ferrite
- removed TP7: TestPoint_Hole1, 4ms_TestPoint:TestPoint_WireHole, symbol MG_ELECTROMECANICAL:TestPoint_Hole1
- added C41: 220uF, EasyEDA:CAP-SMD_BD10.0-L10.3-W10.3-LS11.3-FD, symbol easyeda2kicad:UUD1H221MNL1GS
- added C46: 100uF, EasyEDA:CAP-SMD_BD8.0-L8.3-W8.3-FD, symbol EasyEDA:RVT1H101M0810-C72480
- added D1: MBRA340T, Diode_SMD_AKL:D_SMA, symbol Diode_Schottky_AKL:MBRA340T
- added D2: 1N5819HW-7-F, EasyEDA:SOD-123_L2.7-W1.6-LS3.7-RD, symbol EasyEDA:1N5819HW-7-F
- added JP1: (no value), SparkFun-Jumper:Jumper_2_NO, symbol SparkFun-Jumper:SolderJumper_2_Open
- added L1: APH0630T4R7M, EasyEDA:IND-SMD_L7.0-W6.6_APH0630, symbol easyeda2kicad:APH0630T4R7M
- added TP12: TestPoint_Hole1, 4ms_TestPoint:TestPoint_WireHole, symbol MG_ELECTROMECANICAL:TestPoint_Hole1
Connections:
- net +3.3V: now also JP1.2 (B); no longer C44.1, C45.1, D3.A, U3.1 (FB)
- net +5V: now also D2.2 (A)
- net GND: now also C41.2, C46.2
- net VCC_IN: now also D1.2 (A)
- net sw: now also L1.1
- net vdc_in renamed VDC
- net VDC: now also C41.1, C46.1, D1.1 (K), D2.1 (K)
- new net ps_out: C44.1, C45.1, D3.A, JP1.1 (A), L1.2, TP12.1, U3.1 (FB)
Other:
- note added: "Entrada 5V a 32V"
- moved on the sheet: C1, C2, TP6
