File: PLC4UNI-GC1_PCB/control.kicad_sch (KiCad schematic)
At the start: 22 parts, among them J1 Conn_02x08_Odd_Even, SW1 TS-1088-AR02016, U1 ESP32-S3-WROOM-1, U10 ADS1115IDGS, U4 RS485-PROTECT

Commit message: Actualizacion a la fecha
Parts:
- removed C25: 100nf, Capacitor_SMD_AKL:C_0603_1608Metric, symbol Capacitor_AKL:C_0603
- removed D17: ESD5Z3.3T, Diode_SMD_AKL:D_SOD-523, symbol Diode_TVS_AKL:ESD5Z3.3T
- removed U1: ESP32-S3-WROOM-1, RF_Module:ESP32-S3-WROOM-1U, symbol RF_Module:ESP32-S3-WROOM-1
- removed U4: RS485-PROTECT, MG_footprints:RS-485-PROTECT, symbol MG_CONNECTORS:RS485-PROTECT
- added D17: SMBJ12CA, Diode_SMD_AKL:D_SMB_TVS, symbol Diode_TVS_AKL:SMBJ12CA
- added D23, D24: SMBJ6.5CA, Diode_SMD_AKL:D_SMB_TVS, symbol Diode_TVS_AKL:SMBJ6.5CA
- added R73, R74, R75: 0R, Resistor_SMD_AKL:R_0603_1608Metric, symbol Resistor_US_AKL:R_0603
- added R76, R77: 1K, Resistor_SMD_AKL:R_0603_1608Metric, symbol Resistor_US_AKL:R_0603
- added SW2: TS-1088-AR02016, EasyEDA:SW-SMD_L3.9-W3.0-P4.45, symbol EasyEDA:TS-1088-AR02016
- added U1: TD301M485_C5451847, EasyEDA:COMM-TH_TD301M485, symbol EasyEDA:TD301M485_C5451847
- added U19: ESP32-S3-WROOM-1, Espressif:ESP32-S3-WROOM-1U, symbol Espressif:ESP32-S3-WROOM-1
- R30, R31: value R_0603 -> 10K; LCSC Part # (none) -> C844918
- R4: value 22K -> 1K
Connections:
- net +24V is gone; now on net +3.3V: R30.1
- net i2c_scl is gone; now on net I2C_SCK: U10.10 (SCL)
- net i2c_sda is gone; now on net I2C_SDA: U10.9 (SDA)
- net +3.3V: now also R31.1, R4.1, R73.1, U1.4 (VCC), U19.2 (3V3); no longer R4.2
- net CON_RS485_A: now also D17.1 (K), D23.2 (A), R76.1, U1.7 (B)
- net CON_RS485_B: now also D17.2 (A), D24.2 (A), R77.2, U1.6 (A)
- net CON_RS485_G: now also D23.1 (K), D24.1 (K), R76.2, U1.5 (RGND)
- net EMRX: now also U19.36 (U0RXD/GPIO44/CLK_OUT2)
- net EM_TX: now also U19.37 (U0TXD/GPIO43/CLK_OUT1)
- net EN: now also R4.2, U19.3 (EN); no longer R4.1, SW1.1
- net GND: now also SW1.1, SW2.1, U1.3 (GND), U19.1 (GND), U19.40 (GND), U19.41 (GND); no longer R31.2, SW1.2
- net I2C_SCK: now also U19.11 (GPIO18/U1RXD/ADC2_CH7/CLK_OUT3)
- net I2C_SDA: now also U19.10 (GPIO17/U1TXD/ADC2_CH6)
- net IN_NPN1: now also SW1.2, U19.27 (GPIO0/BOOT)
- net IN_NPN2: now also U19.39 (GPIO1/TOUCH1/ADC1_CH0)
- net IN_NPN3: now also U19.38 (GPIO2/TOUCH2/ADC1_CH1)
- net IN_NPN4: now also U19.15 (GPIO3/TOUCH3/ADC1_CH2)
- net IN_PNP1: now also SW2.2, U19.16 (GPIO46)
- net IN_PNP2: now also U19.24 (GPIO47/SPICLK_P/SUBSPICLK_P_DIFF)
- net LCD_CS: now also J1.7 (Pin_7), U19.35 (MTMS/GPIO42); no longer J1.13 (Pin_13)
- net LCD_EN: now also J1.4 (Pin_4), R73.2; no longer J1.12 (Pin_12)
- net LED_INFO: now also U19.26 (GPIO45)
- net OUT-PNP/st1: now also R74.2
- net OUT-PNP/st2: now also R75.2
- net OUT_NPN1: now also U19.4 (GPIO4/TOUCH4/ADC1_CH3)
- net OUT_NPN2: now also U19.5 (GPIO5/TOUCH5/ADC1_CH4)
- net OUT_NPN3: now also U19.6 (GPIO6/TOUCH6/ADC1_CH5)
- net OUT_NPN4: now also U19.7 (GPIO7/TOUCH7/ADC1_CH6)
- net OUT_PNP1: now also U19.8 (GPIO15/U0RTS/ADC2_CH4/XTAL_32K_P)
- net OUT_PNP2: now also U19.9 (GPIO16/U0CTS/ADC2_CH5/XTAL_32K_N)
- net OUT_RLY1: now also U19.23 (GPIO21)
- net OUT_RLY2: now also U19.31 (GPIO38/FSPIWP/SUBSPIWP)
- net RESET: now also J1.5 (Pin_5), U19.22 (GPIO14/TOUCH14/ADC2_CH3/FSPIWP/FSPIDQS/SUBSPIWP); no longer J1.11 (Pin_11)
- net RS485-RX: now also R30.2, U1.1 (RXD), U19.12 (GPIO8/TOUCH8/ADC1_CH7/SUBSPICS1)
- net RS485-TX: now also R31.2, U1.2 (TXD), U19.17 (GPIO9/TOUCH9/ADC1_CH8/FSPIHD/SUBSPIHD)
- net SD_CS: now also U19.18 (GPIO10/TOUCH10/ADC1_CH9/FSPICS0/FSPIIO4/SUBSPICS0)
- net SPI_CLK: now also J1.13 (Pin_13), U19.20 (GPIO12/TOUCH12/ADC2_CH1/FSPICLK/FSPIIO6/SUBSPICLK); no longer J1.9 (Pin_9)
- net SPI_MISO: now also J1.9 (Pin_9), U19.21 (GPIO13/TOUCH13/ADC2_CH2/FSPIQ/FSPIIO7/SUBSPIQ); no longer J1.7 (Pin_7)
- net SPI_MOSI: now also J1.11 (Pin_11), U19.19 (GPIO11/TOUCH11/ADC2_CH0/FSPID/FSPIIO5/SUBSPID); no longer J1.5 (Pin_5)
- net TEMP_CS: now also U19.25 (GPIO48/SPICLK_N/SUBSPICLK_N_DIFF)
- net TP_INT: now also J1.6 (Pin_6), U19.33 (MTDO/GPIO40/CLK_OUT2); no longer J1.14 (Pin_14)
- net USB+: now also J1.14 (Pin_14), U19.14 (GPIO20/U1CTS/ADC2_CH9/CLK_OUT1/USB_D+); no longer J1.4 (Pin_4)
- net USB-: now also J1.12 (Pin_12), U19.13 (GPIO19/U1RTS/ADC2_CH8/CLK_OUT2/USB_D-); no longer J1.6 (Pin_6)
- removed net IN_VDC_ADC: R30.2, R31.1
- new net: R77.1, U1.8 (VO)
- new net ST1_ST2: R74.1, R75.1, U19.32 (MTCK/GPIO39/CLK_OUT3/SUBSPICS1)
- new net TC_FAULT: U19.34 (MTDI/GPIO41/CLK_OUT1)
- no-connect marks 3 -> 0
Other:
- company: (none) -> ITLA
- title: (none) -> PLC4UNI NIVARA-GC1
- moved on the sheet: C26, D18, D19, D20, D21, J1, LED5, R50, SW1
